File: Pico/pico_watering_system/pico_watering_system.kicad_pcb (KiCad board)
At the start: 2 copper layers, 97.8 x 66 mm, 33 parts, among them J1 P1, J2 P2, J3 s1, J4 s2, J5 IN, J6 Water level sensor 1, J7 Water level sensor 2, Q1 IRFZ44N, Q2 IRFZ44N, U1 pi pico, U2 L7805, U3 tact_switch, U4 tact_switch

Commit message: after milling
Parts:
- PI PICO: renamed from U1
- renumbered J1 to P1, J2 to P2, J3 to S1, J4 to S2, J5 to VIN, J6 to WL1, J7 to WL2
Routing:
- net LED_G2: track 16.8 -> 17.3 mm
Other:
- board text added: "+ -"
- board text added: "- 3V3 S1"
- board text added: "- 3V3 S2"
- board text added: "- S"
- board text added: "NIKODEM BARTNIK"
